Commit message: Underconstruction_URDF

File: urdf/solar_urdf2.urdf (robot description, URDF)
Before this commit: robot solar_urdf2, 9 links, 8 joints
Links:
- link TEEN1: geometry collision mesh filename=package://transporter_description/meshes/TEEN1.STL; visual mesh filename=package://transporter_description/meshes/TEEN1.STL
- link TEEN2: geometry collision mesh filename=package://transporter_description/meshes/TEEN2.STL; visual mesh filename=package://transporter_description/meshes/TEEN2.STL
- link TEEN3: geometry collision mesh filename=package://transporter_description/meshes/TEEN3.STL; visual mesh filename=package://transporter_description/meshes/TEEN3.STL
- link TEEN4: geometry collision mesh filename=package://transporter_description/meshes/TEEN4.STL; visual mesh filename=package://transporter_description/meshes/TEEN4.STL
- link WHEEL1: geometry collision mesh filename=package://transporter_description/meshes/WHEEL1.STL; visual mesh filename=package://transporter_description/meshes/WHEEL1.STL
- link WHEEL2: geometry collision mesh filename=package://transporter_description/meshes/WHEEL2.STL; visual mesh filename=package://transporter_description/meshes/WHEEL2.STL
- link WHEEL3: geometry collision mesh filename=package://transporter_description/meshes/WHEEL3.STL; visual mesh filename=package://transporter_description/meshes/WHEEL3.STL
- link WHEEL4: geometry collision mesh filename=package://transporter_description/meshes/WHEEL4.STL; visual mesh filename=package://transporter_description/meshes/WHEEL4.STL
- link base_link: geometry collision mesh filename=package://transporter_description/meshes/base_link.STL; visual mesh filename=package://transporter_description/meshes/base_link.STL
Joints:
- joint WHEEL1: limit lower=1E+15 upper=1E+15 effort=1E+15 velocity=1E+15 -> lower=1E-15 upper=1E+15 effort=1E+15 velocity=1E+15
- joint WHEEL2: limit lower=1E+15 upper=1E+15 effort=1E+15 velocity=1E+15 -> lower=1E-15 upper=1E+15 effort=1E+15 velocity=1E+15
- joint WHEEL3: limit lower=1E+15 upper=1E+15 effort=1E+15 velocity=1E+15 -> lower=1E-15 upper=1E+15 effort=1E+15 velocity=1E+15
- joint WHEEL4: limit lower=1E+15 upper=1E+15 effort=1E+15 velocity=1E+15 -> lower=1E-15 upper=1E+15 effort=1E+15 velocity=1E+15

Commit message: Add Description

File: urdf/solar_urdf2.urdf (robot description, URDF)
Before this commit: robot transporter_description, 9 links, 8 joints
Joints:
- joint WHEEL1: type revolute -> continuous
- joint WHEEL2: type revolute -> continuous
- joint WHEEL3: type revolute -> continuous
- joint WHEEL4: type revolute -> continuous

Commit message: edit param

File: urdf/solar_urdf2.urdf (robot description, URDF)
Before this commit: robot transporter_description, 9 links, 8 joints
Links:
- removed link base_link
- added link base_footprint, mass 158.02; collision mesh filename=package://transporter_description/meshes/base_link.STL; visual mesh filename=package://transporter_description/meshes/base_link.STL
- added link gps_link, mass 0.02; collision cylinder length=0.1 radius=0.025; visual cylinder length=0.1 radius=0.025
- added link imu_link, mass 0.01; collision box size=0.05 0.05 0.02; visual box size=0.05 0.05 0.02
Joints:
- added joint gps_joint: type fixed, parent base_footprint, child gps_link, origin xyz=0 0 2.0 rpy=0 0 0
- added joint imu_joint: type fixed, parent base_footprint, child imu_link, origin xyz=0 0 1.0 rpy=0 0 0
- joint TEEN1: parent base_link -> base_footprint
- joint TEEN2: parent base_link -> base_footprint
- joint TEEN3: parent base_link -> base_footprint
- joint TEEN4: parent base_link -> base_footprint
- joint WHEEL1: parent base_link -> base_footprint
- joint WHEEL2: parent base_link -> base_footprint
- joint WHEEL3: parent base_link -> base_footprint
- joint WHEEL4: parent base_link -> base_footprint
